File: canton3/canton3.sch (KiCad schematic (older format))
At the start: 25 parts, among them J1 Conn_01x18, Q1 PN2222A, Q2 PN2222A, Q3 PN2222A, Q4 PN2222A, U1 LM317_TO220, U2 CJMCU-4080, U3 ModuleDRV8833

Commit message: pcb canton3
Parts:
- removed Q4: PN2222A, Package_TO_SOT_THT:TO-92_Inline, symbol Transistor_BJT:PN2222A
- removed R10: 2200, Resistor_THT:R_Axial_DIN0207_L6.3mm_D2.5mm_P7.62mm_Horizontal, symbol Device:R
- removed R6: R, Resistor_THT:R_Axial_DIN0207_L6.3mm_D2.5mm_P7.62mm_Horizontal, symbol Device:R
- removed U2: CJMCU-4080, Module:module_1x8, symbol DBN:CJMCU-4080
- added J1: Conn_01x03_Female, Connector_PinHeader_2.54mm:PinHeader_1x03_P2.54mm_Vertical, symbol Connector:Conn_01x03_Female
- added R1: 680, Resistor_THT:R_Axial_DIN0207_L6.3mm_D2.5mm_P7.62mm_Horizontal, symbol Device:R
- J1: value Conn_01x18 -> Conn_01x17; footprint Connector_PinHeader_2.54mm:PinHeader_1x18_P2.54mm_Horizontal -> Connector_PinHeader_2.54mm:PinHeader_1x17_P2.54mm_Horizontal; symbol Connector_Generic:Conn_01x18 -> Connector_Generic:Conn_01x17
- R2, R3: value R -> 1000
- R4: value R -> 2200
- R5: value R -> 4700
Connections:
- net labels removed: 3.3V, CT0, ISENSE
- wire segments 96 -> 75
Other:
- moved on the sheet: R30
