File: canton3/canton3.kicad_pcb (KiCad board)
At the start: 2 copper layers, 45.7 x 52.1 mm, 23 parts, among them J1 Conn_01x03_Female, J2 Conn_01x17, Q5 PN2222A, Q6 PN2222A, Q7 PN2222A, U4 LM317_TO220, U6 ModuleDRV8833

Commit message: mainboard3 again
Parts:
- J2: footprint Connector_PinHeader_2.54mm:PinHeader_1x17_P2.54mm_Vertical -> Connector_PinHeader_2.54mm:PinHeader_1x17_P2.54mm_Horizontal
