File: dispatcher/dispatcher.sch (KiCad schematic (older format))
At the start: 29 parts, among them J1 Conn_01x06_Female, J2 Conn_01x18, K1 HFD2_005-S-L2-D, K2 HFD2_005-S-L2-D, U1 INA3221_Module, U2 ULN2803A, U3 ULN2803A, U5 MCP2551-I-P, U6 ChinaBluePill-bluepill-D3_Boa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

Commit message: mainboard3 again
Parts:
- removed C1: CP, Capacitor_THT:C_Disc_D3.4mm_W2.1mm_P2.50mm, symbol Device:CP
- added C? (x2): C, Capacitor_THT:C_Disc_D3.4mm_W2.1mm_P2.50mm, symbol Device:C
Connections:
- wire segments 119 -> 120
Changed lines of the file:
@@
 L power:+5V #PWR0103
 U 1 1 61B365A9
-P 9050 7625
-F 0 "#PWR0103" H 9050 7475 50  0001 C CNN
-F 1 "+5V" H 9065 7798 50  0000 C CNN
-F 2 "" H 9050 7625 50  0001 C CNN
-F 3 "" H 9050 7625 50  0001 C CNN
-	1    9050 7625
+P 9050 7425
+F 0 "#PWR0103" H 9050 7275 50  0001 C CNN
+F 1 "+5V" H 9065 7598 50  0000 C CNN
+F 2 "" H 9050 7425 50  0001 C CNN
+F 3 "" H 9050 7425 50  0001 C CNN
+	1    9050 7425
 	1    0    0    -1
 $EndComp
@@
 $EndComp
 $Comp
-L Device:CP C1
-U 1 1 61C49DD3
-P 6675 6175
-F 0 "C1" V 6420 6175 50  0000 C CNN
-F 1 "CP" V 6511 6175 50  0000 C CNN
-F 2 "Capacitor_THT:C_Disc_D3.4mm_W2.1mm_P2.50mm" H 6713 6025 50  0001 C CNN
-F 3 "~" H 6675 6175 50  0001 C CNN
-	1    6675 6175
-	0    1    1    0
-$EndComp
-$Comp
 L power:GND #PWR0122
 U 1 1 61C4BDE7
@@
 Wire Wire Line
 	6025 7775 6200 7775
+$Comp
+L Device:C C?
+U 1 1 61BD4F6E
+P 9200 7425
+F 0 "C?" V 8948 7425 50  0000 C CNN
+F 1 "C" V 9039 7425 50  0000 C CNN
+F 2 "Capacitor_THT:C_Disc_D3.4mm_W2.1mm_P2.50mm" H 9238 7275 50  0001 C CNN
+F 3 "~" H 9200 7425 50  0001 C CNN
+	1    9200 7425
+	0    1    1    0
+$EndComp
+Wire Wire Line
+	9050 7625 9050 7425
+Connection ~ 9050 7425
+$Comp
+L power:GND #PWR?
+U 1 1 61BDC921
+P 9350 7425
+F 0 "#PWR?" H 9350 7175 50  0001 C CNN
+F 1 "GND" V 9355 7297 50  0000 R CNN
+F 2 "" H 9350 7425 50  0001 C CNN
+F 3 "" H 9350 7425 50  0001 C CNN
+	1    9350 7425
+	0    -1   -1   0
+$EndComp
+$Comp
+L Device:C C?
+U 1 1 61BEA66C
+P 6675 6175
+F 0 "C?" V 6423 6175 50  0000 C CNN
+F 1 "C" V 6514 6175 50  0000 C CNN
+F 2 "Capacitor_THT:C_Disc_D3.4mm_W2.1mm_P2.50mm" H 6713 6025 50  0001 C CNN
+F 3 "~" H 6675 6175 50  0001 C CNN
+	1    6675 6175
+	0    1    1    0
+$EndComp
 $EndSCHEMATC
