File: mainboard3/mainboard3/mainboard3.kicad_pcb (KiCad board)
At the start: 2 copper layers, 27 parts, among them J0 Conn_01x18, J1 Conn_01x18, J2 Conn_01x18, J3 Conn_01x18, J4 Conn_01x18, J5 Conn_01x18, T0 Screw_Terminal_01x06, T1 Screw_Terminal_01x06, T10 Screw_Terminal_01x06, T11 Screw_Terminal_01x06, T12 Screw_Terminal_01x06, T2 Screw_Terminal_01x06, T3 Screw_Terminal_01x06, T4 Screw_Terminal_01x06, T5 Screw_Terminal_01x06, T6 Screw_Terminal_01x06, T7 Screw_Terminal_01x06, T8 Screw_Terminal_01x06, T9 Screw_Terminal_01x06, U1 STM32_F4xx, U2 ModuleINA3221, U3 ModuleINA3221, U4 ModuleINA3221, U5 ModuleINA3221, U6 ULN2803A, U7 ULN2803A, X1 Screw_Terminal_01x04

Commit message: adding CAN interface
Parts:
- moved X1 99.5 mm to (268.0, 29.2)
- moved U5 41.9 mm to (115.6, 146.7)
- moved U4 39.4 mm to (133.3, 146.7)
- moved U2 36.9 mm to (166.4, 146.7)
- moved U3 36.9 mm to (149.9, 146.7)
- moved U7 31.4 mm to (228.0, 129.5)
- moved T9 28.4 mm to (204.5, 149.9)
- moved T8 27.3 mm to (223.5, 149.9)
- moved J5 25.4 mm to (48.3, 94.0)
- moved U6 25.3 mm to (260.4, 129.5)
- moved T12 23.0 mm to (50.8, 114.3)
- moved T6 21.8 mm to (260.4, 149.9)
- moved T7 21.8 mm to (242.6, 149.9)
- moved T4 16.7 mm to (76.2, 114.3)
- moved J4 16.6 mm to (73.7, 94.0)
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Routing:
- net 12Vunreg: track 488.5 -> 127.0 mm
- net VSENSE4_0: track 178.9 -> 32.8 mm
- net ETR1: track 139.3 -> 0.00 mm, vias 1 -> 0
- net Net-(J4-Pad8): track 0.00 -> 125.8 mm
- net TURN7A: track 107.5 -> 0.00 mm
- net TURN7B: track 104.4 -> 0.00 mm
- net TURN5B: track 104.0 -> 0.00 mm
- net CT2_2: track 102.3 -> 0.00 mm
- net CT2_3: track 101.6 -> 0.00 mm
- net VSENSE4_1: track 199.5 -> 99.9 mm
- net CT2_1: track 98.2 -> 0.00 mm
- net I2C3_SCL: track 89.4 -> 0.00 mm
- net I2C3_SDA: track 88.8 -> 0.00 mm
- net 3V3: track 80.4 -> 0.00 mm
- net PWM5_1: track 225.8 -> 154.4 mm, vias 1 -> 0
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
Commit message: mainboard3 again
Parts:
- removed T0, T1, T12, T2, T3, T4: Screw_Terminal_01x06, Connector_PinHeader_2.54mm:PinHeader_1x06_P2.54mm_Vertical
- added 10k1: R, Resistor_THT:R_Axial_DIN0207_L6.3mm_D2.5mm_P7.62mm_Horizontal, F.Cu at (251.5, 55.9)
- added C1: 100nF, Capacitor_THT:C_Disc_D3.4mm_W2.1mm_P2.50mm, F.Cu at (87.6, 166.4)
- added C2: 100nF, Capacitor_THT:C_Disc_D3.4mm_W2.1mm_P2.50mm, F.Cu at (245.1, 61.0)
- added C3: 100nF, Capacitor_THT:C_Disc_D3.4mm_W2.1mm_P2.50mm, F.Cu at (223.5, 61.0)
- added C4: 100nF, Capacitor_THT:C_Disc_D3.4mm_W2.1mm_P2.50mm, F.Cu at (194.3, 61.0)
- added C5: 100nF, Capacitor_THT:C_Disc_D3.4mm_W2.1mm_P2.50mm, F.Cu at (180.3, 61.0)
- added C6: 0.1µF, Capacitor_THT:C_Disc_D3.4mm_W2.1mm_P2.50mm, F.Cu at (53.3, 177.8)
- added C7: 10µF, Capacitor_THT:CP_Radial_Tantal_D5.0mm_P2.50mm, F.Cu at (47.0, 170.2)
- added J6: Conn_01x06_Female, Connector_PinHeader_2.54mm:PinHeader_1x06_P2.54mm_Vertical, F.Cu at (73.7, 170.2)
- added J7: Conn_01x02_Female, Connector_PinHeader_2.54mm:PinHeader_1x02_P2.54mm_Vertical, F.Cu at (336.6, 232.4)
- added JG2: Conn_01x03_Female, Connector_PinHeader_2.54mm:PinHeader_1x03_P2.54mm_Vertical, F.Cu at (243.8, 66.0)
- added JG3: Conn_01x03_Female, Connector_PinHeader_2.54mm:PinHeader_1x03_P2.54mm_Vertical, F.Cu at (222.2, 66.0)
- added JG4: Conn_01x03_Female, Connector_PinHeader_2.54mm:PinHeader_1x03_P2.54mm_Vertical, F.Cu at (196.8, 67.3)
- added JG5: Conn_01x03_Female, Connector_PinHeader_2.54mm:PinHeader_1x03_P2.54mm_Vertical, F.Cu at (171.4, 64.8)
- added JI2: Conn_01x06_Female, Connector_PinHeader_2.54mm:PinHeader_1x06_P2.54mm_Vertical, F.Cu at (233.7, 40.6)
- added JI3: Conn_01x06_Female, Connector_PinHeader_2.54mm:PinHeader_1x06_P2.54mm_Vertical, F.Cu at (210.8, 40.6)
- added JI4: Conn_01x06_Female, Connector_PinHeader_2.54mm:PinHeader_1x06_P2.54mm_Vertical, F.Cu at (180.3, 40.6)
- added JI5: Conn_01x06_Female, Connector_PinHeader_2.54mm:PinHeader_1x06_P2.54mm_Vertical, F.Cu at (156.2, 40.6)
- added JLED1: Conn_01x08_Female, Connector_PinHeader_2.54mm:PinHeader_1x08_P2.54mm_Vertical, F.Cu at (287.0, 157.5)
- added JLED2: Conn_01x08_Female, Connector_PinHeader_2.54mm:PinHeader_1x08_P2.54mm_Vertical, F.Cu at (312.4, 246.4)
- added JP1: Jumper, Connector_PinHeader_2.54mm:PinHeader_1x02_P2.54mm_Vertical, F.Cu at (71.1, 163.8)
- added JT_0_1: Screw_Terminal_01x02, Connector_PinHeader_2.54mm:PinHeader_1x02_P2.54mm_Vertical, F.Cu at (241.3, -14.0)
- added JT_0_2: Screw_Terminal_01x02, Connector_PinHeader_2.54mm:PinHeader_1x02_P2.54mm_Vertical, F.Cu at (241.3, -5.08)
- added JT_0_3: Screw_Terminal_01x02, Connector_PinHeader_2.54mm:PinHeader_1x02_P2.54mm_Vertical, F.Cu at (241.3, 3.81)
- added JT_1_1: Screw_Terminal_01x02, Connector_PinHeader_2.54mm:PinHeader_1x02_P2.54mm_Vertical, F.Cu at (252.7, 3.81)
- added JT_1_2: Screw_Terminal_01x02, Connector_PinHeader_2.54mm:PinHeader_1x02_P2.54mm_Vertical, F.Cu at (252.7, -5.08)
- added JT_1_3: Screw_Terminal_01x02, Connector_PinHeader_2.54mm:PinHeader_1x02_P2.54mm_Vertical, F.Cu at (252.7, -14.0)
- added JT_2_1: Screw_Terminal_01x02, Connector_PinHeader_2.54mm:PinHeader_1x02_P2.54mm_Vertical, F.Cu at (265.4, 3.81)
- added JT_2_2: Screw_Terminal_01x02, Connector_PinHeader_2.54mm:PinHeader_1x02_P2.54mm_Vertical, F.Cu at (265.4, -5.08)
- added JT_3_1: Screw_Terminal_01x02, Connector_PinHeader_2.54mm:PinHeader_1x02_P2.54mm_Vertical, F.Cu at (265.4, -14.0)
- added JT_3_2: Screw_Terminal_01x02, Connector_PinHeader_2.54mm:PinHeader_1x02_P2.54mm_Vertical, F.Cu at (252.7, 14.0)
- added JT_4_1: Screw_Terminal_01x02, Connector_PinHeader_2.54mm:PinHeader_1x02_P2.54mm_Vertical, F.Cu at (265.4, 14.0)
- added JT_5_1: Screw_Terminal_01x02, Connector_PinHeader_2.54mm:PinHeader_1x02_P2.54mm_Vertical, F.Cu at (241.3, 14.0)
- added R1: R, Resistor_THT:R_Axial_DIN0207_L6.3mm_D2.5mm_P7.62mm_Horizontal, F.Cu at (68.6, 185.4)
- added R10: 10k, Resistor_THT:R_Axial_DIN0207_L6.3mm_D2.5mm_P7.62mm_Horizontal, F.Cu at (167.6, 54.6)
- added R11: 10k, Resistor_THT:R_Axial_DIN0207_L6.3mm_D2.5mm_P7.62mm_Horizontal, F.Cu at (170.2, 54.6)
- added R12: 10k, Resistor_THT:R_Axial_DIN0207_L6.3mm_D2.5mm_P7.62mm_Horizontal, F.Cu at (172.7, 54.6)
- added R13: 10k, Resistor_THT:R_Axial_DIN0207_L6.3mm_D2.5mm_P7.62mm_Horizontal, F.Cu at (189.2, 53.3)
- added R14: 10k, Resistor_THT:R_Axial_DIN0207_L6.3mm_D2.5mm_P7.62mm_Horizontal, F.Cu at (191.8, 53.3)
- added R15: 10k, Resistor_THT:R_Axial_DIN0207_L6.3mm_D2.5mm_P7.62mm_Horizontal, F.Cu at (194.3, 53.3)
- added R16: 10k, Resistor_THT:R_Axial_DIN0207_L6.3mm_D2.5mm_P7.62mm_Horizontal, F.Cu at (214.6, 53.3)
- added R17: 10k, Resistor_THT:R_Axial_DIN0207_L6.3mm_D2.5mm_P7.62mm_Horizontal, F.Cu at (237.5, 53.3)
- added R18: 10k, Resistor_THT:R_Axial_DIN0207_L6.3mm_D2.5mm_P7.62mm_Horizontal, F.Cu at (186.7, 53.3)
- added R19: 10k, Resistor_THT:R_Axial_DIN0207_L6.3mm_D2.5mm_P7.62mm_Horizontal, F.Cu at (172.7, 57.1)
- added R2: 120, Resistor_THT:R_Axial_DIN0207_L6.3mm_D2.5mm_P7.62mm_Horizontal, F.Cu at (68.6, 174.0)
- added R20: R, Resistor_THT:R_Axial_DIN0207_L6.3mm_D2.5mm_P7.62mm_Horizontal, F.Cu at (289.6, 191.8)
- added R21: R, Resistor_THT:R_Axial_DIN0207_L6.3mm_D2.5mm_P7.62mm_Horizontal, F.Cu at (289.6, 189.2)
- added R22: R, Resistor_THT:R_Axial_DIN0207_L6.3mm_D2.5mm_P7.62mm_Horizontal, F.Cu at (289.6, 186.7)
- added R23: R, Resistor_THT:R_Axial_DIN0207_L6.3mm_D2.5mm_P7.62mm_Horizontal, F.Cu at (289.6, 184.2)
- added R24: R, Resistor_THT:R_Axial_DIN0207_L6.3mm_D2.5mm_P7.62mm_Horizontal, F.Cu at (289.6, 181.6)
- added R25: R, Resistor_THT:R_Axial_DIN0207_L6.3mm_D2.5mm_P7.62mm_Horizontal, F.Cu at (289.6, 179.1)
- added R26: R, Resistor_THT:R_Axial_DIN0207_L6.3mm_D2.5mm_P7.62mm_Horizontal, F.Cu at (289.6, 176.5)
- added R27: R, Resistor_THT:R_Axial_DIN0207_L6.3mm_D2.5mm_P7.62mm_Horizontal, F.Cu at (289.6, 174.0)
- added R28: 510, Resistor_THT:R_Axial_DIN0207_L6.3mm_D2.5mm_P7.62mm_Horizontal, F.Cu at (41.9, 181.2)
- added R29: 200, Resistor_THT:R_Axial_DIN0207_L6.3mm_D2.5mm_P7.62mm_Horizontal, F.Cu at (52.1, 180.3)
- added R3: 10k, Resistor_THT:R_Axial_DIN0207_L6.3mm_D2.5mm_P7.62mm_Horizontal, F.Cu at (217.2, 53.3)
- added R30: 240, Resistor_THT:R_Axial_DIN0207_L6.3mm_D2.5mm_P7.62mm_Horizontal, F.Cu at (49.5, 184.2)
- added R4: 10k, Resistor_THT:R_Axial_DIN0207_L6.3mm_D2.5mm_P7.62mm_Horizontal, F.Cu at (219.7, 53.3)
- added R5: 10k, Resistor_THT:R_Axial_DIN0207_L6.3mm_D2.5mm_P7.62mm_Horizontal, F.Cu at (222.2, 53.3)
- added R6: 10k, Resistor_THT:R_Axial_DIN0207_L6.3mm_D2.5mm_P7.62mm_Horizontal, F.Cu at (240.0, 53.3)
- added R7: 10k, Resistor_THT:R_Axial_DIN0207_L6.3mm_D2.5mm_P7.62mm_Horizontal, F.Cu at (242.6, 53.3)
- added R8: 10k, Resistor_THT:R_Axial_DIN0207_L6.3mm_D2.5mm_P7.62mm_Horizontal, F.Cu at (245.1, 53.3)
- added R9: 10k, Resistor_THT:R_Axial_DIN0207_L6.3mm_D2.5mm_P7.62mm_Horizontal, F.Cu at (251.5, 58.4)
- added SW1: SW_DIP_x01, Connector_PinHeader_2.54mm:PinHeader_1x02_P2.54mm_Vertical, F.Cu at (38.1, 170.2)
- added U10: LM317_TO220, Package_TO_SOT_THT:TO-220-3_Vertical, F.Cu at (44.0, 177.1)
- added U8: MCP2551-I-P, Package_DIP:DIP-8_W7.62mm, F.Cu at (76.2, 189.2)
- added U9: ULN2803A, Package_DIP:DIP-18_W7.62mm, F.Cu at (193.0, 208.3)
- moved X1 206.4 mm to (321.3, 228.6), turned to 180 degrees
- moved T9 134.2 mm to (321.3, 215.9), turned to 180 degrees
- moved U1 127.6 mm to (109.2, 78.7), turned to 90 degrees
- moved U2 117.2 mm to (248.9, 63.5)
- moved U3 112.8 mm to (226.1, 63.5)
- moved U6 107.8 mm to (160.0, 90.2), turned to 0 degrees
- moved U4 105.4 mm to (198.1, 63.5)
- moved U5 103.1 mm to (176.5, 63.5)
- moved T8 102.4 mm to (321.3, 180.3), turned to 180 degrees
- moved J0 89.5 mm to (231.1, 24.1)
- moved J1 87.9 mm to (203.2, 24.1)
- moved J2 86.4 mm to (175.3, 24.1)
- moved J3 84.9 mm to (147.3, 24.1)
- moved J4 83.5 mm to (119.4, 24.1)
- moved J5 80.8 mm to (88.9, 24.1)
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Connections:
- net LED1 renamed BOARD_LED
- net LED2 renamed BOARD_LED2
- net SWO renamed Net-(U1-Pad17)
- net usb_dm renamed Net-(U1-Pad31)
- net usb_dp renamed Net-(U1-Pad32)
- J0 pad 2: TRACK0_1 -> I1A
- J1 pad 2: TRACK1_1 -> I4A
- J2 pad 2: TRACK2_1 -> I7A
- J3 pad 2: TRACK3_1 -> I12A
- J4 pad 2: TRACK4_1 -> I11A
- J5 pad 2: TRACK5_1 -> I10A
- T6 pad 2: GND -> 12Vunreg
- T6 pad 5: GND -> 12Vunreg
- T7 pad 2: GND -> 12Vunreg
- T7 pad 5: GND -> 12Vunreg
- T8 pad 2: GND -> 12Vunreg
- T8 pad 5: GND -> 12Vunreg
- T9 pad 2: GND -> 12Vunreg
- T9 pad 5: GND -> 12Vunreg
- U1 pad 11: TURN8A -> TURN6A
- U1 pad 13: TIM_OUT -> CAN_RX
- U1 pad 14: TURN1B -> CAN_TX
- U1 pad 18: TURN2B -> TURN4B
- U1 pad 29: R5 -> Net-(U1-Pad29)
- U1 pad 33: R1 -> _TURN1B
- U1 pad 34: R2 -> Net-(U1-Pad34)
- U1 pad 39: CT2_3 -> CT0_1
- U1 pad 41: ROT2 -> Net-(U1-Pad41)
- U1 pad 42: CT2_2 -> CT0_2
- U1 pad 43: CT2_1 -> CT0_3
- U1 pad 44: ROT1 -> Net-(U1-Pad44)
- U1 pad 59: CT0_2 -> CT5_2
- U1 pad 60: CT0_3 -> CT5_3
- U1 pad 61: CT0_1 -> CT5_1
- U1 pad 62: TURN4A -> TURN2B
- U1 pad 64: TURN4B -> TURN6B
- U1 pad 65: VSENSE0_1 -> VSENSE5_1
- U1 pad 66: VSENSE0_0 -> VSENSE5_0
- U1 pad 67: VSENSE5_1 -> VSENSE4_0
- U1 pad 71: VSENSE1_0 -> VSENSE3_0
- U1 pad 72: VSENSE1_1 -> VSENSE3_1
- U1 pad 73: VSENSE2_0 -> VSENSE0_0
- U1 pad 74: VSENSE2_1 -> VSENSE0_1
- U1 pad 75: VSENSE3_0 -> VSENSE2_0
- U1 pad 76: VSENSE3_1 -> VSENSE2_1
- U1 pad 80: VSENSE5_0 -> VSENSE1_0
- U1 pad 82: VSENSE4_0 -> VSENSE1_1
- U1 pad 83: CT5_1 -> CT2_3
- U1 pad 84: ETR1 -> Net-(U1-Pad84)
- U1 pad 85: CT5_2 -> CT2_2
- U1 pad 87: CT5_3 -> CT2_1
- U1 pad 92: TURN6B -> TURN2A
- U1 pad 93: TURN1A -> TURN1B
- U1 pad 96: TURN2A -> TURN1A
Routing:
- net CT1_3: track 0.00 -> 192.9 mm, vias 0 -> 1
- net I2C3_SDA: track 0.00 -> 177.1 mm
- net I2C3_SCL: track 0.00 -> 171.7 mm
- net CT5_1: track 241.5 -> 72.8 mm
- net TRACK5_0: track 20.3 -> 180.8 mm, vias 0 -> 1
- net CT5_3: track 233.1 -> 73.1 mm
- net CT5_2: track 233.1 -> 73.7 mm
- net 3V3: track 0.00 -> 157.9 mm
- net VSENSE5_1: track 202.7 -> 52.9 mm
- net VSENSE5_0: track 194.0 -> 47.7 mm
- net CT1_2: track 52.7 -> 191.3 mm, vias 0 -> 1
- net TRACK4_0: track 20.3 -> 154.9 mm
- net CT1_1: track 40.0 -> 174.1 mm, vias 0 -> 1
- net I9B: track 0.00 -> 130.0 mm, vias 0 -> 1
- net CT0_1: track 94.4 -> 222.8 mm, vias 0 -> 1
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
Commit message: mainboard3  routing
Parts:
- removed J6: Conn_01x06_Female, Connector_PinHeader_2.54mm:PinHeader_1x06_P2.54mm_Vertical
- removed JLED1, JLED2: Conn_01x08_Female, Connector_PinHeader_2.54mm:PinHeader_1x08_P2.54mm_Vertical
- removed T6, T7, T8, T9: Screw_Terminal_01x06, Connector_PinHeader_2.54mm:PinHeader_1x06_P2.54mm_Vertical
- added C8: 0.1µF, Capacitor_THT:C_Disc_D3.4mm_W2.1mm_P2.50mm, F.Cu at (213.4, 112.4)
- added C9: 10µF, Capacitor_THT:CP_Radial_Tantal_D5.0mm_P2.50mm, F.Cu at (209.6, 111.1)
- added J8: Conn_02x05_Odd_Even, Connector_PinHeader_2.54mm:PinHeader_2x05_P2.54mm_Vertical, F.Cu at (255.3, 102.2)
- added J_BUS1: Conn_01x05_Female, Connector_PinHeader_2.54mm:PinHeader_1x05_P2.54mm_Vertical, F.Cu at (214.0, -19.7)
- added J_GUI1: Conn_01x05_Female, Connector_PinHeader_2.54mm:PinHeader_1x05_P2.54mm_Vertical, F.Cu at (87.6, 73.0)
- added J_T1: Conn_01x03_Female, Connector_PinHeader_2.54mm:PinHeader_1x03_P2.54mm_Vertical, F.Cu at (213.4, 86.4)
- added J_T2: Conn_01x03_Female, Connector_PinHeader_2.54mm:PinHeader_1x03_P2.54mm_Vertical, F.Cu at (213.4, 74.9)
- added J_T3: Conn_01x03_Female, Connector_PinHeader_2.54mm:PinHeader_1x03_P2.54mm_Vertical, F.Cu at (228.6, 86.4)
- added J_T4: Conn_01x03_Female, Connector_PinHeader_2.54mm:PinHeader_1x03_P2.54mm_Vertical, F.Cu at (228.6, 74.9)
- added J_T5: Conn_01x03_Female, Connector_PinHeader_2.54mm:PinHeader_1x03_P2.54mm_Vertical, F.Cu at (245.1, 86.4)
- added J_T6: Conn_01x03_Female, Connector_PinHeader_2.54mm:PinHeader_1x03_P2.54mm_Vertical, F.Cu at (257.8, 86.4)
- added J_T7: Conn_01x03_Female, Connector_PinHeader_2.54mm:PinHeader_1x03_P2.54mm_Vertical, F.Cu at (257.8, 74.9)
- added SW2: SW_DIP_x01, Connector_PinHeader_2.54mm:PinHeader_1x02_P2.54mm_Vertical, F.Cu at (232.4, 118.7)
- added SW3: SW_DIP_x01, Connector_PinHeader_2.54mm:PinHeader_1x02_P2.54mm_Vertical, F.Cu at (224.2, 118.7)
- added U11: LM317_TO220, Package_TO_SOT_THT:TO-220-3_Vertical, F.Cu at (206.9, 117.5)
- R27: value R -> 240
- moved T11 283.3 mm to (-15.2, 86.4)
- moved T5 265.6 mm to (15.2, 80.6)
- moved T10 170.5 mm to (91.4, 122.6), turned to 90 degrees
- moved R30 153.9 mm to (188.6, 118.1), turned to 90 degrees
- moved J7 147.5 mm to (242.6, 118.7), turned to 270 degrees
- moved U10 147.1 mm to (178.4, 117.5)
- moved C6 146.8 mm to (184.8, 112.4)
- moved C7 146.4 mm to (181.0, 111.1), turned to 180 degrees
- moved R28 145.2 mm to (173.4, 119.4), turned to 90 degrees
- moved R29 136.0 mm to (169.5, 111.8)
- moved SW1 134.7 mm to (162.6, 118.7), turned to 270 degrees
- moved U9 122.5 mm to (204.5, 86.4)
- moved R26 112.1 mm to (198.1, 111.8), turned to 270 degrees
- moved R25 106.0 mm to (201.9, 119.4), turned to 90 degrees
- moved R20 97.5 mm to (249.6, 102.9)
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Connections:
- net LED6 renamed Net-(U9-Pad6)
- net LED7 renamed Net-(U9-Pad7)
- net LED8 renamed Net-(U9-Pad8)
- net Net-(U1-Pad17) renamed SWO
- net Net-(U1-Pad31) renamed usb_dm
- net Net-(U1-Pad32) renamed usb_dp
- net TURN8A renamed Net-(U7-Pad7)
- C1 pad 2: +5V -> 5V
- J0 pad 17: 12Vunreg -> 12V
- J1 pad 17: 12Vunreg -> 12V
- J2 pad 17: 12Vunreg -> 12V
- J3 pad 17: 12Vunreg -> 12V
- J4 pad 17: 12Vunreg -> 12V
- J5 pad 17: 12Vunreg -> 12V
- J7 pad 2: 12Vunreg -> Net-(J7-Pad2)
- R20 pad 1: 5V -> Net-(J8-Pad2)
- R20 pad 2: Net-(JLED1-Pad1) -> 5V
- R21 pad 1: 5V -> Net-(J8-Pad4)
- R21 pad 2: Net-(JLED1-Pad3) -> 5V
- R22 pad 1: 5V -> Net-(J8-Pad6)
- R22 pad 2: Net-(JLED1-Pad5) -> 5V
- R23 pad 1: 5V -> Net-(J8-Pad8)
- R23 pad 2: Net-(JLED1-Pad7) -> 5V
- R24 pad 1: 5V -> Net-(J8-Pad10)
- R24 pad 2: Net-(JLED2-Pad1) -> 5V
- R25 pad 1: 5V -> Net-(R25-Pad1)
- R25 pad 2: Net-(JLED2-Pad3) -> Net-(R25-Pad2)
- R26 pad 1: 5V -> Net-(R25-Pad2)
- R26 pad 2: Net-(JLED2-Pad5) -> GND
- R27 pad 1: 5V -> Net-(C9-Pad1)
- R27 pad 2: Net-(JLED2-Pad7) -> Net-(R25-Pad1)
- SW1 pad 2: V5 -> 5V
- U1 pad 11: TURN6A -> TURN2A
- U1 pad 12: TURN8B -> TURN2B
- U1 pad 18: TURN4B -> TURN1A
- U1 pad 19: TURN3A -> TURN8B
- U1 pad 20: TURN3B -> TURN1B
- U1 pad 27: TURN7A -> TURN5A
- U1 pad 29: Net-(U1-Pad29) -> TURN6B
- U1 pad 30: TURN7B -> TURN6A
- U1 pad 33: _TURN1B -> TURN7A
- U1 pad 34: Net-(U1-Pad34) -> TURN7B
- U1 pad 39: CT0_1 -> PWM5_2
- U1 pad 41: Net-(U1-Pad41) -> ROT2
- U1 pad 42: CT0_2 -> PWM5_1
- U1 pad 44: Net-(U1-Pad44) -> ROT1
- U1 pad 47: PWM5_1 -> LED2
- U1 pad 62: TURN2B -> TURN3A
- U1 pad 63: TURN5A -> LED4
- U1 pad 64: TURN6B -> CT0_2
- U1 pad 79: TURN6A -> LED3
- U1 pad 84: Net-(U1-Pad84) -> CT0_1
- U1 pad 92: TURN2A -> TURN3B
- U1 pad 93: TURN1B -> TURN4A
- U1 pad 95: PWM5_2 -> LED1
- U1 pad 96: TURN1A -> TURN4B
- U6 pad 10: 12Vunreg -> 12V
- U7 pad 10: 12Vunreg -> 12V
- U7 pad 8: TURN8B -> Net-(U7-Pad8)
- U8 pad 3: +5V -> 5V
- U9 pad 5: LED5 -> BOARD_LED2
- X1 pad 1: 12Vunreg -> 12V
Routing:
- net 12V: track 0.00 -> 577.9 mm, vias 0 -> 1
- net 5V: track 0.00 -> 490.7 mm
- net Net-(J_BUS1-Pad4): track 0.00 -> 314.7 mm, vias 0 -> 1
- net 3V3: track 157.9 -> 458.3 mm, vias 0 -> 1
- net Net-(JP1-Pad1): track 0.00 -> 292.4 mm, vias 0 -> 1
- net PWM5_2: track 99.0 -> 216.0 mm, vias 2 -> 1
- net Net-(J_T6-Pad1): track 0.00 -> 110.7 mm
- net LED4: track 0.00 -> 108.9 mm, vias 0 -> 1
- net Net-(J_T7-Pad1): track 0.00 -> 105.1 mm
- net Net-(J_T6-Pad3): track 0.00 -> 105.1 mm
- net Net-(J_T7-Pad3): track 0.00 -> 101.4 mm
- net Net-(J_T4-Pad1): track 0.00 -> 100.8 mm
- net Net-(J_T4-Pad3): track 0.00 -> 98.1 mm
- net Net-(J_T5-Pad1): track 0.00 -> 97.9 mm
- net LED3: track 0.00 -> 94.7 mm, vias 0 -> 2
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- added copper zone on B.Cu, net GND

Commit message: before moving to kicad6
Parts:
- moved J_BUS1 284.4 mm to (297.8, 252.1), turned to 180 degrees
- moved J8 172.7 mm to (102.2, 22.2)
- moved J5 167.0 mm to (233.7, 107.3), turned to 0 degrees
- moved J7 158.7 mm to (86.4, 146.7), turned to 180 degrees
- moved R20 152.7 mm to (118.7, 24.1), turned to 0 degrees
- moved R21 152.7 mm to (118.7, 26.7), turned to 0 degrees
- moved R22 152.4 mm to (118.7, 29.8), turned to 0 degrees
- moved R23 152.4 mm to (118.7, 32.4), turned to 0 degrees
- moved R24 152.0 mm to (118.7, 35.6), turned to 0 degrees
- moved SW2 147.1 mm to (86.4, 136.5), turned to 0 degrees
- moved SW3 138.1 mm to (86.4, 128.3), turned to 0 degrees
- moved R27 129.4 mm to (92.1, 149.2), turned to 0 degrees
- moved C8 120.6 mm to (97.2, 144.8), turned to 0 degrees
- moved U9 120.0 mm to (92.1, 44.5), turned to 90 degrees
- moved J4 118.1 mm to (203.2, 107.3), turned to 0 degrees
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Connections:
- U1 pad 43: CT0_3 -> TURN3A
- U1 pad 45: CT1_3 -> CT5_3
- U1 pad 46: CT1_2 -> CT5_2
- U1 pad 48: CT1_1 -> CT5_1
- U1 pad 59: CT5_2 -> CT1_2
- U1 pad 60: CT5_3 -> CT1_3
- U1 pad 61: CT5_1 -> CT1_1
- U1 pad 62: TURN3A -> CT0_3
- U1 pad 75: VSENSE2_0 -> VSENSE1_0
- U1 pad 76: VSENSE2_1 -> VSENSE1_1
- U1 pad 80: VSENSE1_0 -> VSENSE2_0
- U1 pad 82: VSENSE1_1 -> VSENSE2_1
Routing:
- net 5V: track 490.7 -> 193.3 mm
- net Net-(J_BUS1-Pad4): track 314.7 -> 28.8 mm, vias 1 -> 0
- net Net-(JP1-Pad1): track 292.4 -> 26.6 mm, vias 1 -> 0
- net 12V: track 577.9 -> 330.5 mm, vias 1 -> 0
- net 3V3: track 458.3 -> 265.8 mm, vias 1 -> 0
- net TRACK5_0: track 180.8 -> 52.5 mm
- net VSENSE5_0: track 47.7 -> 170.0 mm
- net VSENSE5_1: track 52.9 -> 169.4 mm
- net Net-(J_T6-Pad1): track 110.7 -> 0.00 mm
- net PWM5_2: track 216.0 -> 105.6 mm, vias 1 -> 0
- net PWM3_2: track 152.0 -> 44.1 mm, vias 1 -> 0
- net GND: track 44.3 -> 150.1 mm, vias 11 -> 0
- net Net-(J_T7-Pad1): track 105.1 -> 0.00 mm
- net Net-(J_T6-Pad3): track 105.1 -> 0.00 mm
- net PWM3_1: track 152.4 -> 49.3 mm, vias 1 -> 0
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- removed copper zone on B.Cu, net GND
