File: Mainboard4/CurrentDetect4/CurrentDetect4.kicad_pcb (KiCad board)
At the start: 2 copper layers, 62.9 x 180 mm, 38 parts, among them J1 Conn_01x04_Male, J2 Conn_01x12_Male, U1 INA3221_Module, U2 INA3221_Module, U3 INA3221_Module, U4 INA3221_Module

Commit message: nearly ok
Parts:
- added REF**: MountingHole_2.2mm_M2, MountingHole:MountingHole_2.2mm_M2, F.Cu at (113.0, 182.9)
- moved R2 10.4 mm to (116.6, 25.4)
- moved R3 10.4 mm to (114.0, 25.4)
- moved R1 9.35 mm to (110.0, 21.6), turned to 0 degrees
- moved REF** 5.08 mm to (156.8, 57.1)
Routing:
- net 3V3: track 313.4 -> 327.0 mm
- net I12B: track 110.0 -> 104.9 mm
- net I12A: track 53.3 -> 48.3 mm
- net I1B: track 37.8 -> 41.8 mm
- net Net-(R3-Pad2): track 19.8 -> 23.6 mm
- net Net-(R2-Pad2): track 19.8 -> 23.6 mm

Commit message: mainboard4 ready for production
Parts:
- R13: renamed from 10k1; value R13 -> 10k
- moved C3 40.4 mm to (120.9, 137.7)
- moved R9 40.4 mm to (105.6, 130.1)
- moved JT_2_1 40.4 mm to (80.8, 104.7)
- moved JT_3_2 40.4 mm to (80.8, 133.2)
- moved R8 40.4 mm to (108.1, 130.1)
- moved C2 40.4 mm to (120.9, 91.3)
- moved C4 40.4 mm to (120.9, 184.0)
- moved J1 40.4 mm to (137.8, 209.2)
- moved R12 40.4 mm to (105.6, 176.4)
- moved R13 40.4 mm to (105.4, 44.7)
- moved R6 40.4 mm to (105.6, 83.7)
- moved R7 40.4 mm to (110.7, 130.1)
- moved REF** 40.4 mm to (133.3, 179.4)
- moved U1 40.4 mm to (123.4, 48.7)
- moved U2 40.4 mm to (123.4, 95.7)
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Other:
- board text added: "Z-ATC CurrentDetect v0.4 © Daniel Braun 2022"
