File: Mainboard4/CurrentDetect4/CurrentDetect4.kicad_sch (KiCad schematic)
At the start: 36 parts, among them J1 Conn_01x04_Male, J2 Conn_01x12_Male, U1 INA3221_Module, U2 INA3221_Module, U3 INA3221_Module, U4 INA3221_Module

Commit message: mainboard4 ready for production
Parts:
- R13: renamed from 10k1; value R13 -> 10k
Changed lines of the file:
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@@
   (symbol (lib_id "Device:R") (at 45.72 170.815 90) (unit 1)
     (in_bom yes) (on_board yes)
-    (property "Reference" "10k1" (id 0) (at 50.165 168.275 90))
-    (property "Value" "R13" (id 1) (at 45.085 171.45 90))
+    (property "Reference" "R13" (id 0) (at 50.165 168.275 90))
+    (property "Value" "10k" (id 1) (at 45.085 171.45 90))
     (property "Footprint" "Resistor_THT:R_Axial_DIN0207_L6.3mm_D2.5mm_P7.62mm_Horizontal" (id 2) (at 45.72 172.593 90)
       (effects (font (size 1.27 1.27)) hide)
@@
       (reference "#PWR0109") (unit 1) (value "GND") (footprint "")
     )
-    (path "/07df0eaa-99e0-41ed-af52-7fb22b9b0201"
-      (reference "10k1") (unit 1) (value "R13") (footprint "Resistor_THT:R_Axial_DIN0207_L6.3mm_D2.5mm_P7.62mm_Horizontal")
-    )
     (path "/f9efb531-936d-4192-a4d7-9aaeec9d7799"
       (reference "C1") (unit 1) (value "100nF") (footprint "Capacitor_THT:C_Disc_D3.4mm_W2.1mm_P2.50mm")
@@
       (reference "R12") (unit 1) (value "10k") (footprint "Resistor_THT:R_Axial_DIN0207_L6.3mm_D2.5mm_P7.62mm_Horizontal")
     )
+    (path "/07df0eaa-99e0-41ed-af52-7fb22b9b0201"
+      (reference "R13") (unit 1) (value "10k") (footprint "Resistor_THT:R_Axial_DIN0207_L6.3mm_D2.5mm_P7.62mm_Horizontal")
+    )
     (path "/b229243d-11d5-4a2d-a522-e20d99107088"
