File: Mainboard4/Mainboard4/Mainboard4.kicad_sch (KiCad schematic)
At the start: 43 parts, among them J0 Conn_01x18, J1 Conn_01x18, J2 Conn_01x18, J3 Conn_01x18, J4 Conn_01x18, J5 Conn_01x18, J7 Conn_01x02_Female, J8 Conn_01x12_Female, SW1 SW_DIP_x01, SW2 SW_DIP_x01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

Commit message: nearly ok
Parts:
- removed C3: 10µF, Capacitor_THT:CP_Radial_Tantal_D5.0mm_P2.50mm, symbol Device:C
- removed C?: 10µF, Capacitor_THT:CP_Radial_Tantal_D5.0mm_P2.50mm, symbol Device:CP
- removed C?: 0.1µF, Capacitor_THT:C_Disc_D3.4mm_W2.1mm_P2.50mm, symbol Device:CP
- removed J_I2C_3: Conn_01x04_Female, Connector_PinHeader_2.54mm:PinHeader_1x04_P2.54mm_Vertical, symbol Connector:Conn_01x04_Female
- added C3, C5: 10µF, Capacitor_THT:CP_Radial_Tantal_D5.0mm_P2.50mm, symbol Device:C_Polarized
- added C4: 0.1µF, Capacitor_THT:CP_Radial_Tantal_D5.0mm_P2.50mm, symbol Device:C_Polarized
- added J6: Conn_02x08_Odd_Even, Connector_PinHeader_2.54mm:PinHeader_2x08_P2.54mm_Vertical, symbol Connector_Generic:Conn_02x08_Odd_Even
- added JP3, JP4: Jumper_2_Open, Connector_PinHeader_2.54mm:PinHeader_1x02_P2.54mm_Vertical, symbol Jumper:Jumper_2_Open
- added J_I2C_3: Conn_01x06_Female, Connector_PinHeader_2.54mm:PinHeader_1x06_P2.54mm_Vertical, symbol Connector:Conn_01x06_Female
- added R10, R11, R12, R13, R14, R15, R16, R17: R, Resistor_THT:R_Axial_DIN0207_L6.3mm_D2.5mm_P7.62mm_Horizontal, symbol Device:R
- added U7: ULN2803A, Package_DIP:DIP-18_W7.62mm, symbol Transistor_Array:ULN2803A
- renumbered J7 to J_POWER1
Connections:
- net 12V: now also J_GUI1.1 (Pin_1), JP3.2 (B), JP4.2 (B); no longer SW3.2
- net 12Vunreg: now also C4.1, JP4.1 (A)
- net 3V3: now also J_I2C_3.4 (Pin_4)
- net 5V: now also R10.2, R11.2, R12.2, R13.2, R14.2, R15.2, R16.2, R17.2, U7.10 (COM)
- net BOARD_LED2: now also U7.7 (I7)
- net GND: now also C3.2, C4.2, C5.2, J_I2C_3.3 (Pin_3), U7.9 (GND)
- net I2C3_SCL: now also J_I2C_3.1 (Pin_1)
- net I2C3_SDA: now also J_I2C_3.2 (Pin_2)
- net LED1: now also U2.48 (PD8), U7.1 (I1)
- net LED2: now also U2.92 (PE15), U7.2 (I2)
- net LED3: now also U2.87 (PE12), U7.3 (I3); no longer U2.79 (PC5)
- net LED4: now also U2.85 (PE10), U7.4 (I4); no longer U2.63 (PC13)
- net ROT1: now also J_I2C_3.5 (Pin_5)
- net ROT2: now also J_I2C_3.6 (Pin_6)
- net at J_BUS1.4 (Pin_4), J_GUI1.4 (Pin_4), R8.1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: now also R9.2; no longer R9.1
- net at JP1.1 (A), J_BUS1.5 (Pin_5), J_GUI1.5 (Pin_5)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: now also JP2.2 (B); no longer JP2.1 (A)
- net at R6.1, SW3.1, U3.2 (VO): now also C5.1
- net at R3.1, SW1.1, U1.2 (VO): now also C3.1
- net LED5: now reaches U2.83 (PE8)
- net LED5: now also U7.5 (I5)
- new net: J6.6 (Pin_6), R12.1
- new net: J6.10 (Pin_10), R14.1
- new net: J6.16 (Pin_16), R17.1
- new net: J6.2 (Pin_2), R10.1
- new net: JP2.1 (A), R9.1
- new net: J6.14 (Pin_14), R16.1
- new net: J6.15 (Pin_15), U7.11 (O8)
- new net: J6.13 (Pin_13), U7.12 (O7)
- new net: J6.11 (Pin_11), U7.13 (O6)
- new net: J6.9 (Pin_9), U7.14 (O5)
- new net: J6.7 (Pin_7), U7.15 (O4)
- new net: J6.5 (Pin_5), U7.16 (O3)
- new net: J6.3 (Pin_3), U7.17 (O2)
- new net: J6.1 (Pin_1), U7.18 (O1)
- new net: J6.8 (Pin_8), R13.1
- new net: JP3.1 (A), SW3.2
- new net: J6.4 (Pin_4), R11.1
- new net: J6.12 (Pin_12), R15.1
- new net LED6: U2.79 (PC5), U7.6 (I6)
- new net LED8: U2.63 (PC13), U7.8 (I8)
Other:
- moved on the sheet: C1, C2, JP1, JP2, J_BUS1, J_GUI1, J_I2C_1, J_POWER1, J_T1, J_T2, J_T3, J_T4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

Commit message: nearly ok
Changed lines of the file:
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@@
     )
   )
-  (global_label "5V" (shape input) (at 379.73 89.535 180) (fields_autoplaced)
+  (global_label "5V" (shape input) (at 382.27 89.535 180) (fields_autoplaced)
     (effects (font (size 1.27 1.27)) (justify right))
-    (property "Intersheet References" "${INTERSHEET_REFS}" (id 0) (at 128.905 -5.08 0)
+    (property "Intersheet References" "${INTERSHEET_REFS}" (id 0) (at 131.445 -5.08 0)
       (effects (font (size 1.27 1.27)) hide)
     )

Commit message: ..
Connections:
- net 5V: now also C3.1, R3.1, SW1.1, U1.2 (VO); no longer C1.2, SW1.2, U2.49 (5V), U2.50 (5V), U2.51 (5V), U2.52 (5V), U4.3 (VDD)
- new net 5VCPU: C1.2, SW1.2, U2.49 (5V), U2.50 (5V), U2.51 (5V), U2.52 (5V), U4.3 (VDD)
Other:
- moved on the sheet: SW1
Changed lines of the file:
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@@
   (junction (at 361.315 165.735) (diameter 0) (color 0 0 0 0)
   )
+  (junction (at 66.675 88.265) (diameter 0) (color 0 0 0 0)
+  )
+  (junction (at 361.315 175.895) (diameter 0) (color 0 0 0 0)
+  )
+  (junction (at 489.585 267.335) (diameter 0) (color 0 0 0 0)
+  )
+  (junction (at 116.205 88.265) (diameter 0) (color 0 0 0 0)
+  )
+  (junction (at 535.94 267.335) (diameter 0) (color 0 0 0 0)
+  )
+  (junction (at 498.475 160.02) (diameter 0) (color 0 0 0 0)
+  )
+  (junction (at 343.535 281.94) (diameter 0) (color 0 0 0 0)
+  )
+  (junction (at 328.295 269.24) (diameter 0) (color 0 0 0 0)
+  )
+  (junction (at 384.175 111.125) (diameter 0) (color 0 0 0 0)
+  )
   (junction (at 374.015 269.24) (diameter 0) (color 0 0 0 0)
   )
-  (junction (at 66.675 88.265) (diameter 0) (color 0 0 0 0)
-  )
-  (junction (at 361.315 175.895) (diameter 0) (color 0 0 0 0)
-  )
-  (junction (at 489.585 267.335) (diameter 0) (color 0 0 0 0)
-  )
-  (junction (at 116.205 88.265) (diameter 0) (color 0 0 0 0)
-  )
-  (junction (at 535.94 267.335) (diameter 0) (color 0 0 0 0)
-  )
-  (junction (at 498.475 160.02) (diameter 0) (color 0 0 0 0)
-  )
-  (junction (at 343.535 281.94) (diameter 0) (color 0 0 0 0)
-  )
-  (junction (at 328.295 269.24) (diameter 0) (color 0 0 0 0)
-  )
-  (junction (at 384.175 111.125) (diameter 0) (color 0 0 0 0)
-  )
   (junction (at 81.915 88.265) (diameter 0) (color 0 0 0 0)
   )
   (junction (at 361.315 170.815) (diameter 0) (color 0 0 0 0)
   )
+  (junction (at 379.095 269.24) (diameter 0) (color 0 0 0 0)
+  )
   (junction (at 69.215 88.265) (diameter 0) (color 0 0 0 0)
   )
@@
     (stroke (width 0) (type default) (color 0 0 0 0))
   )
-  (wire (pts (xy 389.255 269.24) (xy 408.94 269.24))
-    (stroke (width 0) (type default) (color 0 0 0 0))
-  )
   (wire (pts (xy 535.94 267.335) (xy 535.94 275.59))
     (stroke (width 0) (type default) (color 0 0 0 0))
@@
     (stroke (width 0) (type default) (color 0 0 0 0))
   )
+  (wire (pts (xy 374.015 269.24) (xy 379.095 269.24))
+    (stroke (width 0) (type default) (color 0 0 0 0))
+  )
   (wire (pts (xy 57.785 154.305) (xy 51.435 154.305))
     (stroke (width 0) (type default) (color 0 0 0 0))
@@
     (stroke (width 0) (type default) (color 0 0 0 0))
   )
-  (wire (pts (xy 408.94 263.525) (xy 408.94 269.24))
-    (stroke (width 0) (type default) (color 0 0 0 0))
-  )
   (wire (pts (xy 87.63 51.435) (xy 93.345 51.435))
     (stroke (width 0) (type default) (color 0 0 0 0))
@@
     (stroke (width 0) (type default) (color 0 0 0 0))
   )
+  (wire (pts (xy 379.095 262.89) (xy 379.095 269.24))
+    (stroke (width 0) (type default) (color 0 0 0 0))
+  )
   (polyline (pts (xy 304.165 67.31) (xy 419.735 67.31))
     (stroke (width 0) (type default) (color 0 0 0 0))
@@
     (stroke (width 0) (type default) (color 0 0 0 0))
   )
+  (wire (pts (xy 379.095 269.24) (xy 380.365 269.24))
+    (stroke (width 0) (type default) (color 0 0 0 0))
+  )
   (wire (pts (xy 377.825 108.585) (xy 377.825 121.285))
     (stroke (width 0) (type default) (color 0 0 0 0))
@@
     (stroke (width 0) (type default) (color 0 0 0 0))
   )
+  (wire (pts (xy 408.94 269.24) (xy 408.94 263.525))
+    (stroke (width 0) (type default) (color 0 0 0 0))
+  )
   (wire (pts (xy 362.585 281.94) (xy 343.535 281.94))
+    (stroke (width 0) (type default) (color 0 0 0 0))
+  )
+  (wire (pts (xy 395.605 269.24) (xy 408.94 269.24))
     (stroke (width 0) (type default) (color 0 0 0 0))
   )
@@
     )
   )
-  (global_label "5V" (shape input) (at 345.44 82.55 90) (fields_autoplaced)
-    (effects (font (size 1.27 1.27)) (justify left))
-    (property "Intersheet References" "${INTERSHEET_REFS}" (id 0) (at 128.905 -5.08 0)
-      (effects (font (size 1.27 1.27)) hide)
+  (global_label "5VCPU" (shape input) (at 345.44 82.55 90) (fields_autoplaced)
+    (effects (font (size 1.27 1.27)) (justify left))
+    (property "Intersheet References" "${INTERSHEET_REFS}" (id 0) (at 345.3606 73.9683 90)
+      (effects (font (size 1.27 1.27)) (justify left) hide)
     )
   )
@@
     )
   )
-  (global_label "5V" (shape output) (at 408.94 263.525 90) (fields_autoplaced)
-    (effects (font (size 1.27 1.27)) (justify left))
-    (property "Intersheet References" "${INTERSHEET_REFS}" (id 0) (at -24.13 226.06 0)
-      (effects (font (size 1.27 1.27)) hide)
+  (global_label "5VCPU" (shape output) (at 408.94 263.525 90) (fields_autoplaced)
+    (effects (font (size 1.27 1.27)) (justify left))
+    (property "Intersheet References" "${INTERSHEET_REFS}" (id 0) (at 408.8606 254.9433 90)
+      (effects (font (size 1.27 1.27)) (justify left) hide)
     )
   )
@@
     )
   )
-  (global_label "5V" (shape input) (at 98.425 83.185 90) (fields_autoplaced)
-    (effects (font (size 1.27 1.27)) (justify left))
-    (property "Intersheet References" "${INTERSHEET_REFS}" (id 0) (at 5.08 -102.87 0)
-      (effects (font (size 1.27 1.27)) hide)
+  (global_label "5VCPU" (shape input) (at 98.425 83.185 90) (fields_autoplaced)
+    (effects (font (size 1.27 1.27)) (justify left))
+    (property "Intersheet References" "${INTERSHEET_REFS}" (id 0) (at 98.3456 74.6033 90)
+      (effects (font (size 1.27 1.27)) (justify left) hide)
     )
   )
@@
     (property "Intersheet References" "${INTERSHEET_REFS}" (id 0) (at 99.6156 202.801 90)
       (effects (font (size 1.27 1.27)) (justify right) hide)
+    )
+  )
+  (global_label "5V" (shape output) (at 379.095 262.89 90) (fields_autoplaced)
+    (effects (font (size 1.27 1.27)) (justify left))
+    (property "Intersheet References" "${INTERSHEET_REFS}" (id 0) (at -53.975 225.425 0)
+      (effects (font (size 1.27 1.27)) hide)
     )
   )
@@
     (pin "1")
   )
-  (symbol (lib_id "Switch:SW_DIP_x01") (at 381.635 269.24 0) (unit 1)
+  (symbol (lib_id "Switch:SW_DIP_x01") (at 387.985 269.24 0) (unit 1)
     (in_bom yes) (on_board yes)
-    (property "Reference" "SW1" (id 0) (at 381.635 262.4582 0))
-    (property "Value" "SW_DIP_x01" (id 1) (at 381.635 264.7696 0))
-    (property "Footprint" "Connector_PinHeader_2.54mm:PinHeader_1x02_P2.54mm_Vertical" (id 2) (at 381.635 269.24 0)
-      (effects (font (size 1.27 1.27)) hide)
-    )
-    (property "Datasheet" "~" (id 3) (at 381.635 269.24 0)
-      (effects (font (size 1.27 1.27)) hide)
-    )
+    (property "Reference" "SW1" (id 0) (at 387.985 262.4582 0))
+    (property "Value" "SW_DIP_x01" (id 1) (at 387.985 264.7696 0))
+    (property "Footprint" "Connector_PinHeader_2.54mm:PinHeader_1x02_P2.54mm_Vertical" (id 2) (at 387.985 269.24 0)
+      (effects (font (size 1.27 1.27)) hide)
+    )
+    (property "Datasheet" "~" (id 3) (at 387.985 269.24 0)
+      (effects (font (size 1.27 1.27)) hide)
+    )

Commit message: mainboard4 ready for production
Parts:
- renumbered J6 to J6_LEDS1, J_I2C_3 to J_I2C_3_IUI1, SW3 to SW_12V1, SW1 to SW_5VCPU1, SW2 to SW_GEN1
Connections:
- net 12V: now also SW_12V1.2; no longer JP3.2 (B), JP4.2 (B)
- net at C5.1, R6.1, U3.2 (VO): now also JP3.1 (A); no longer SW_12V1.1
- new net: JP3.2 (B), JP4.2 (B), SW_12V1.1
Other:
- moved on the sheet: C1, C4, C5, JP1, JP2, JP3, JP4, J_BUS1, J_GUI1, J_POWER1, R4, R5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

Commit message: updated to have full USB and external flash
Parts:
- removed R17: R, Resistor_THT:R_Axial_DIN0207_L6.3mm_D2.5mm_P7.62mm_Horizontal, symbol Device:R
Connections:
- net BOARD_LED: now also U5.7 (I7)
- net BOARD_LED2: now also U5.8 (I8); no longer U7.7 (I7)
- net LED6: no longer U2.79 (PC5)
- net TURN2A: now also U2.25 (PD0); no longer U2.18 (PB5)
- net TURN3A: now also U2.63 (PC13); no longer U2.25 (PD0)
- net TURN5B: now also U2.47 (PB15); no longer U2.33 (PA9)
- net TURN6A: now also U2.30 (PC10); no longer U2.34 (PA10)
- net TURN6B: now also U2.28 (PC12); no longer U2.47 (PB15)
- net VSENSE3_0: now also U2.66 (PC0); no longer U2.82 (PB0)
- net VSENSE3_1: now also U2.65 (PC1); no longer U2.66 (PC0)
- net VSENSE4_0: now also U2.68 (PC2); no longer U2.65 (PC1)
- net VSENSE4_1: now also U2.67 (PC3); no longer U2.68 (PC2)
- net VSENSE5_0: now also U2.80 (PC4); no longer U2.67 (PC3)
- net VSENSE5_1: now also U2.79 (PC5); no longer U2.80 (PC4)
- net at U7.11 (O8): no longer J6_LEDS1.15 (Pin_15)
- net LED8: no longer names the net of U7.8 (I8)
- net LED8: no longer U2.63 (PC13)
- net SWO renamed SWO_SPI1_SCK
- removed net TURN4A: U2.28 (PC12), U5.7 (I7)
- removed net TURN4B: U2.30 (PC10), U5.8 (I8)
- new net LED7: U7.7 (I7)
- new net SPI1_MOSI: U2.18 (PB5)
- new net flash_cs: U2.82 (PB0)
- new net usb_otg_id: U2.34 (PA10)
- new net usb_vbus: U2.33 (PA9)
