File: G4/G4_ShieldCurrent/G4_ShieldCurrent.kicad_pcb (KiCad board)
At the start: 2 copper layers, 71.1 x 83.2 mm, 20 parts, among them J1 Conn_01x12_Female, J4 Conn_02x10_Odd_Even, J6 Conn_01x01_Female, U1 INA3221_Module, U2 NUCLEO-G491RE, U3 INA3221_Module

Commit message: misc update
Parts:
- U2: footprint G4Lib:MODULE_NUCLEO-G491RE20 -> G4Lib:MODULE_NUCLEO-G491RE
- moved R1 58.0 mm to (128.3, 104.1), turned to -90 degrees
- moved R2 51.7 mm to (127.6, 93.3), turned to -90 degrees
- moved R10 38.3 mm to (128.3, 121.9), turned to 90 degrees
- moved U3 31.3 mm to (97.2, 139.1), turned to 180 degrees
- moved R3 29.9 mm to (149.2, 139.1)
Connections:
- net I5A renamed T4A
- net I6A renamed T5A
- J1 pad 1: TRACK0_1 -> T0C
- J1 pad 10: I5B -> T4B
- J1 pad 11: TRACK3_1 -> T5C
- J1 pad 12: I6B -> T5B
- J1 pad 2: I1B -> T0B
- J1 pad 3: TRACK0_1 -> T1C
- J1 pad 4: I2B -> T1B
- J1 pad 5: TRACK1_1 -> T2C
- J1 pad 6: I3B -> T2B
- J1 pad 7: TRACK1_1 -> T3C
- J1 pad 8: I4B -> T3B
- J1 pad 9: TRACK2_1 -> T4C
- J4 pad 2: RIA -> T0C
- J4 pad 4: RIB -> T0B
- U1 pad 10: I1B -> T0C
- U1 pad 11: I2A -> T1A
- U1 pad 12: I2B -> T1C
- U1 pad 13: I3A -> T2A
- U1 pad 14: I3B -> T2C
- U1 pad 9: I1A -> T0A
- U2 pad CN10_18: (no net) -> unconnected-(U2-PadCN10_18)
- U2 pad CN10_20: GND -> unconnected-(U2-PadCN10_20)
- U2 pad CN10_9: GND -> unconnected-(U2-PadCN10_9)
- U2 pad CN7_31: unconnected-(U2-PadCN7_31) -> GND
- U3 pad 10: I4B -> T3C
- U3 pad 12: I5B -> T4C
- U3 pad 14: I6B -> T5C
- U3 pad 9: I4A -> T3A
Routing:
- net I2C3_SCL: track 0.00 -> 31.5 mm
