File: G4/G4_ShieldCurrent/G4_ShieldCurrent.kicad_sch (KiCad schematic)
At the start: 20 parts, among them J1 Conn_01x12_Female, J4 Conn_02x10_Odd_Even, J6 Conn_01x01_Female, U1 INA3221_Module, U2 NUCLEO-G491RE, U3 INA3221_Module

Commit message: misc update
Connections:
- net I1A is gone; now on net T0A: U1.9 (VIN1-)
- net I2A is gone; now on net T1A: U1.11 (VIN2-)
- net I3A is gone; now on net T2A: U1.13 (VIN3-)
- net I4A is gone; now on net T3A: U3.9 (VIN1-)
- net RIA is gone; now on net T0C: J4.2 (Pin_2)
- net RIB is gone; now on net T0B: J4.4 (Pin_4)
- net GND: now also U2.CN7_31 (PH1)
- net T0B: now also J1.2 (Pin_2)
- net T1B: now also J1.4 (Pin_4)
- net T2B: now also J1.6 (Pin_6)
- net T3B: now also J1.8 (Pin_8)
- net I1B renamed T0C
- net T0C: now also J1.1 (Pin_1); no longer J1.2 (Pin_2)
- net I2B renamed T1C
- net T1C: now also J1.3 (Pin_3); no longer J1.4 (Pin_4)
- net I3B renamed T2C
- net T2C: now also J1.5 (Pin_5); no longer J1.6 (Pin_6)
- net I4B renamed T3C
- net T3C: now also J1.7 (Pin_7); no longer J1.8 (Pin_8)
- net I5A renamed T4A
- net I5B renamed T4B
- net T4B: no longer U3.12 (VIN2+)
- net I6A renamed T5A
- net I6B renamed T5B
- net T5B: no longer U3.14 (VIN3+)
- removed net TRACK0_1: J1.1 (Pin_1), J1.3 (Pin_3)
- removed net TRACK1_1: J1.5 (Pin_5), J1.7 (Pin_7)
- net TRACK2_1 renamed T4C
- net T4C: now also U3.12 (VIN2+)
- net TRACK3_1 renamed T5C
- net T5C: now also U3.14 (VIN3+)
