File: KicadTemplates/G4_template/G4_template.kicad_sch (KiCad schematic)
At the start: 28 parts, among them J1 Conn_01x04_Female, SW1 SW_SPDT, U1 NUCLEO-G491RE, U3 74HC594

Commit message: change i2c1 and i2c3 for better routing
Connections:
- net SER0: now also JP2.1 (A)
- net SER1: now also JP3.1 (A)
- net SER2: now also JP4.1 (A)
- net SER3: now also JP5.1 (A)
- net SPI3_MOSI: now also JP1.1 (A)
Changed lines of the file:
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@@
+    (stroke (width 0) (type default))
+  )
+  (wire (pts (xy 80.01 229.87) (xy 82.55 229.87))
     (stroke (width 0) (type default))
   )
@@
     (stroke (width 0) (type default))
   )
+  (wire (pts (xy 80.01 226.06) (xy 82.55 226.06))
+    (stroke (width 0) (type default))
+  )
   (wire (pts (xy 342.9 35.56) (xy 311.15 35.56))
     (stroke (width 0) (type default))
@@
     (stroke (width 0) (type default))
   )
+  (wire (pts (xy 80.01 222.25) (xy 82.55 222.25))
+    (stroke (width 0) (type default))
+  )
   (wire (pts (xy 149.86 273.05) (xy 158.75 273.05))
     (stroke (width 0) (type default))
@@
     (stroke (width 0) (type default))
   )
+  (wire (pts (xy 80.01 218.44) (xy 82.55 218.44))
+    (stroke (width 0) (type default))
+  )
+  (wire (pts (xy 80.01 214.63) (xy 82.55 214.63))
+    (stroke (width 0) (type default))
+  )
   (wire (pts (xy 164.465 62.865) (xy 164.465 63.5))
     (stroke (width 0) (type default))
@@
     (stroke (width 0) (type default))
   )
-  (text "SSD1306 DISPLAY\n" (at 235.585 38.1 0)
+  (text "SSD1306 DISPLAY\n" (at 163.83 48.26 0)
     (effects (font (size 1.27 1.27)) (justify left bottom))
   )
@@
     (effects (font (size 1.27 1.27)) (justify left bottom))
   )
-  (text "CAN\n" (at 235.585 29.845 0)
-    (effects (font (size 1.27 1.27)) (justify left bottom))
-  )
-  (text "ina3221 i2c\n" (at 165.1 50.8 0)
-    (effects (font (size 1.27 1.27)) (justify left bottom))
-  )
+  (text "CAN\n" (at 340.36 26.035 0)
+    (effects (font (size 1.27 1.27)) (justify left bottom))
+  )
+  (text "ina3221 i2c\n" (at 242.57 34.29 0)
+    (effects (font (size 1.27 1.27)) (justify left bottom))
+  )
